File: analog-synth-1.sch (KiCad schematic (older format))
At the start: 55 parts, among them J1 CONN_02X08, J2 PJ301M-12, J3 PJ301M-12, J4 PJ301M-12, J5 PJ301M-12, Q1 2N3904, Q2 2N3904, Q3 2N3904, Q4 2N3906, Q5 2N3904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

Commit message: Fix VCO tuning rev1.0.13
Connections:
- wire segments 165 -> 212
Changed lines of the file:
@@
 Title "Analog Synth 1"
 Date "2017-07-31"
-Rev "1.0.12"
+Rev "1.0.13"
 Comp ""
 Comment1 ""
@@
 $EndComp
 Wire Wire Line
-	950  1550 1850 1550
+	950  1550 1450 1550
+Wire Wire Line
+	1450 1550 1850 1550
 Connection ~ 1450 1550
 Wire Wire Line
-	950  1650 2050 1650
+	950  1650 1450 1650
+Wire Wire Line
+	1450 1650 2050 1650
 Connection ~ 1450 1650
 Wire Wire Line
-	950  1750 2050 1750
+	950  1750 1450 1750
+Wire Wire Line
+	1450 1750 2050 1750
 Connection ~ 1450 1750
 Wire Wire Line
-	1450 1750 1450 1950
+	1450 1750 1450 1850
+Wire Wire Line
+	1450 1850 1450 1950
 Connection ~ 1450 1850
 Wire Wire Line
@@
 	1450 1850 950  1850
 Wire Wire Line
-	950  2050 1850 2050
+	950  2050 1450 2050
+Wire Wire Line
+	1450 2050 1850 2050
 Connection ~ 1450 2050
 Text GLabel 1550 1050 1    60   Input ~ 0
@@
 	1550 1350 1550 1050
 Wire Wire Line
-	950  1350 1550 1350
+	950  1350 1450 1350
+Wire Wire Line
+	1450 1350 1550 1350
 Wire Wire Line
 	1650 1450 1650 1050
 Wire Wire Line
-	950  1450 1650 1450
+	950  1450 1450 1450
+Wire Wire Line
+	1450 1450 1650 1450
 Connection ~ 1450 1350
 Connection ~ 1450 1450
@@
 	3900 1100 3700 1100
 Wire Wire Line
-	3450 1450 3900 1450
+	3450 1450 3600 1450
+Wire Wire Line
+	3600 1450 3900 1450
 $Comp
 L POT_TRIM RV1
@@
 	4300 2150 4900 2150
 Wire Wire Line
-	4500 1350 5100 1350
+	4500 1350 4900 1350
+Wire Wire Line
+	4900 1350 5100 1350
 Wire Wire Line
 	4900 2300 4150 2300
 Connection ~ 4900 2150
 Wire Wire Line
-	4900 1350 4900 2300
+	4900 1350 4900 2150
+Wire Wire Line
+	4900 2150 4900 2300
 Connection ~ 3600 1450
 Text GLabel 3000 1450 0    60   Input ~ 0
@@
 $EndComp
 Wire Wire Line
-	6550 3600 6800 3600
+	6550 3600 6700 3600
+Wire Wire Line
+	6700 3600 6800 3600
 Wire Wire Line
 	6550 3600 6550 3500
@@
 	8000 2050 8000 1950
 Wire Wire Line
-	7100 2050 8000 2050
+	7100 2050 7550 2050
+Wire Wire Line
+	7550 2050 8000 2050
 Wire Wire Line
 	7100 2050 7100 1950
@@
 	7100 900  7100 1000
 Wire Wire Line
-	7100 1300 7100 1550
+	7100 1300 7100 1400
+Wire Wire Line
+	7100 1400 7100 1550
 $Comp
 L GND #PWR012
@@
 	8450 1900 8450 1750
 Wire Wire Line
-	8300 1750 8950 1750
+	8300 1750 8450 1750
+Wire Wire Line
+	8450 1750 8950 1750
 Text GLabel 6600 1750 0    60   Input ~ 0
 VIN
@@
 	7550 3200 7550 2800
 Wire Wire Line
-	6950 3200 7550 3200
+	6950 3200 7300 3200
+Wire Wire Line
+	7300 3200 7550 3200
 Wire Wire Line
 	7300 3200 7300 2450
@@
 	7100 1400 6050 1400
 Wire Wire Line
-	6050 1400 6050 3100
+	6050 1400 6050 2450
+Wire Wire Line
+	6050 2450 6050 3100
 Wire Wire Line
 	6050 3100 6350 3100
@@
 	8000 1500 8700 1500
 Wire Wire Line
-	8700 1500 8700 2700
+	8700 1500 8700 1950
+Wire Wire Line
+	8700 1950 8700 2700
 Wire Wire Line
 	8700 1950 8950 1950
@@
 	9950 2700 9950 1850
 Wire Wire Line
-	9550 1850 10150 1850
+	9550 1850 9950 1850
+Wire Wire Line
+	9950 1850 10150 1850
 Wire Wire Line
 	9050 2700 9050 2850
@@
 Text Notes 7800 3600 0    157  ~ 0
 Exponential Converter
-Text GLabel 1400 5600 0    60   Input ~ 0
+Text GLabel 1300 5800 0    60   Input ~ 0
 Exp-CV
 $Comp
@@
 	0    1    1    0
 $EndComp
-Wire Wire Line
-	1400 5600 1600 5600
-Connection ~ 1500 5600
 $Comp
 L LM741 U5
@@
 	1900 5600 2000 5600
 Wire Wire Line
-	2000 5500 2000 5750
+	2000 5500 2000 5600
+Wire Wire Line
+	2000 5600 2000 5750
 Wire Wire Line
 	2000 5500 2500 5500
@@
 Connection ~ 2000 5600
 Wire Wire Line
-	2400 4600 2400 5750
+	2400 4600 2400 5300
+Wire Wire Line
+	2400 5300 2400 5750
 Connection ~ 2400 5300
 $Comp
@@
 $EndComp
 Wire Wire Line
-	2000 6800 2400 6800
+	2000 6800 2200 6800
+Wire Wire Line
+	2200 6800 2400 6800
 Wire Wire Line
 	2400 6800 2400 6650
@@
 	2650 4600 2400 4600
 Wire Wire Line
-	2950 4600 3550 4600
+	2950 4600 3400 4600
+Wire Wire Line
+	3400 4600 3550 4600
 Wire Wire Line
 	3400 4600 3400 5400
 Wire Wire Line
-	3100 5400 3950 5400
+	3100 5400 3400 5400
+Wire Wire Line
+	3400 5400 3950 5400
 Text GLabel 3550 4600 2    60   Input ~ 0
 Tri-SMPL
@@
 	3900 6200 4250 6200
 Wire Wire Line
-	3900 5600 3900 6200
+	3900 5600 3900 5750
+Wire Wire Line
+	3900 5750 3900 6200
 Wire Wire Line
 	3900 5600 3950 5600
@@
 	4550 6200 4900 6200
 Wire Wire Line
-	4900 5500 4900 6450
-Wire Wire Line
-	4550 5500 5050 5500
+	4900 5500 4900 6200
+Wire Wire Line
+	4900 6200 4900 6450
+Wire Wire Line
+	4550 5500 4900 5500
+Wire Wire Line
+	4900 5500 5050 5500
 $Comp
 L R R16
@@
 $EndComp
 Wire Wire Line
-	4150 4950 4350 4950
+	4150 4950 4300 4950
+Wire Wire Line
+	4300 4950 4350 4950
 Wire Wire Line
 	4150 4950 4150 5200
@@
 	4150 5850 4150 5800
 Wire Notes Line
-	850  4250 5800 4250
+	750  4250 5800 4250
 Wire Notes Line
 	5800 4250 5800 7500
 Wire Notes Line
-	5800 7500 850  7500
-Wire Notes Line
-	850  7500 850  4250
+	5800 7500 750  7500
+Wire Notes Line
+	750  7500 750  4250
 Text Notes 5000 6950 0    157  ~ 0
 VCO
@@
 	7900 5050 7900 4500
 Wire Wire Line
-	7550 4500 8050 4500
+	7550 4500 7900 4500
+Wire Wire Line
+	7900 4500 8050 4500
 Wire Wire Line
 	6950 5700 6950 6150
@@
 	7900 6150 7900 5600
 Wire Wire Line
-	7550 5600 8050 5600
+	7550 5600 7900 5600
+Wire Wire Line
+	7900 5600 8050 5600
 $Comp
 L GND #PWR021
@@
 $EndComp
 Wire Wire Line
-	4600 1050 4700 1050
+	4600 1050 4650 1050
+Wire Wire Line
+	4650 1050 4700 1050
 Connection ~ 4650 1050
 $Comp
@@
 Connection ~ 6700 3600
 Wire Wire Line
-	7100 3600 7200 3600
+	7100 3600 7150 3600
+Wire Wire Line
+	7150 3600 7200 3600
 Connection ~ 7150 3600
 Wire Wire Line
@@
 	10000 1450 9950 1450
 Wire Wire Line
-	9550 1450 9650 1450
+	9550 1450 9600 1450
+Wire Wire Line
+	9600 1450 9650 1450
 Connection ~ 9600 1450
 $Comp
@@
 $EndComp
 Wire Wire Line
-	10200 5300 10900 5300
+	10200 5300 10400 5300
+Wire Wire Line
+	10400 5300 10650 5300
+Wire Wire Line
+	10650 5300 10900 5300
 Wire Wire Line
 	10200 5300 10200 5250
@@
 C9's value has a drastic\neffect on the VCO's frequency.
 Wire Wire Line
-	2700 5800 2850 5800
+	2700 5800 2750 5800
+Wire Wire Line
+	2750 5800 2850 5800
 Wire Wire Line
 	3550 5750 3500 5750
 Wire Wire Line
-	3500 5300 3500 5850
+	3500 5300 3500 5750
+Wire Wire Line
+	3500 5750 3500 5850
 Wire Wire Line
 	3500 6150 3500 6200
@@
 	3500 4950 3500 5000
 Wire Wire Line
-	9150 1250 9150 1550
+	9150 1250 9150 1450
+Wire Wire Line
+	9150 1450 9150 1550
 Wire Wire Line
 	9250 1450 9150 1450
@@
 	9950 2700 9450 2700
 Wire Wire Line
-	8700 2700 9150 2700
+	8700 2700 9050 2700
+Wire Wire Line
+	9050 2700 9150 2700
 $Comp
 L R R13
@@
 $EndComp
 Wire Wire Line
-	2150 5300 2500 5300
+	2150 5300 2400 5300
+Wire Wire Line
+	2400 5300 2500 5300
 $Comp
 L POT_TRIM RV4
 U 1 1 598CE1E8
-P 1500 5200
-F 0 "RV4" H 1430 5246 50  0000 R CNN
-F 1 "10k" H 1430 5155 50  0000 R CNN
-F 2 "Potentiometers:Potentiometer_Trimmer_Bourns_3296Y" H 1500 5200 50  0001 C CNN
-F 3 "" H 1500 5200 50  0001 C CNN
-	1    1500 5200
+P 1350 5400
+F 0 "RV4" H 1280 5446 50  0000 R CNN
+F 1 "10k" H 1280 5355 50  0000 R CNN
+F 2 "Potentiometers:Potentiometer_Trimmer_Bourns_3296Y" H 1350 5400 50  0001 C CNN
+F 3 "" H 1350 5400 50  0001 C CNN
+	1    1350 5400
 	1    0    0    -1
 $EndComp
@@
 Wire Wire Line
 	2150 5200 2050 5200
-Wire Wire Line
-	1750 5200 1650 5200
-Wire Wire Line
-	1500 5350 1500 5600
 $Comp
 L POT_TRIM RV3
@@
 	1950 4900 1850 4900
 Wire Wire Line
-	1550 4900 1500 4900
-Wire Wire Line
-	1500 4900 1500 5050
+	1350 4900 1550 4900
 Text Notes 3100 3800 0    60   ~ 0
 RV1 is exponential product control.\nRV2 is product control.\nRV3 and RV4 are sum controls.
 Wire Wire Line
-	3600 1450 3600 2150
+	3600 1450 3600 1800
+Wire Wire Line
+	3600 1800 3600 2150
 Wire Wire Line
 	3600 2150 4000 2150
@@
 $EndComp
 Wire Wire Line
-	1150 3450 1150 3900
+	1150 3450 1150 3850
+Wire Wire Line
+	1150 3850 1150 3900
 Wire Wire Line
 	1150 3850 1200 3850
@@
 $EndComp
 Wire Wire Line
-	2850 6750 3750 6750
+	2850 6750 3000 6750
+Wire Wire Line
+	3000 6750 3650 6750
+Wire Wire Line
+	3650 6750 3750 6750
 Connection ~ 3650 6750
 $Comp
@@
 Wire Wire Line
 	2200 3500 2250 3500
+Wire Wire Line
+	1750 5200 1550 5200
+Wire Wire Line
+	1550 5200 1550 5400
+Wire Wire Line
+	1550 5400 1550 5600
+Wire Wire Line
+	1550 5600 1600 5600
+Wire Wire Line
+	1500 5400 1550 5400
+Connection ~ 1550 5400
+Wire Wire Line
+	1350 5550 1350 5800
+Wire Wire Line
+	1350 5800 1300 5800
+Wire Wire Line
+	1350 5250 1350 4900
 $EndSCHEMATC

Commit message: Fix polarized capacitor footprints rev1.0.14
Parts:
- C12, C13, C14: footprint Capacitors_THT:CP_Radial_D6.3mm_P2.50mm -> Capacitors_THT:CP_Radial_D8.0mm_P3.50mm
Connections:
- wire segments 212 -> 168
Changed lines of the file:
@@
 Title "Analog Synth 1"
 Date "2017-07-31"
-Rev "1.0.13"
+Rev "1.0.14"
 Comp ""
 Comment1 ""
@@
 $EndComp
 Wire Wire Line
-	950  1550 1450 1550
-Wire Wire Line
-	1450 1550 1850 1550
+	950  1550 1850 1550
 Connection ~ 1450 1550
 Wire Wire Line
-	950  1650 1450 1650
-Wire Wire Line
-	1450 1650 2050 1650
+	950  1650 2050 1650
 Connection ~ 1450 1650
 Wire Wire Line
-	950  1750 1450 1750
-Wire Wire Line
-	1450 1750 2050 1750
+	950  1750 2050 1750
 Connection ~ 1450 1750
 Wire Wire Line
-	1450 1750 1450 1850
-Wire Wire Line
-	1450 1850 1450 1950
+	1450 1750 1450 1950
 Connection ~ 1450 1850
 Wire Wire Line
@@
 	1450 1850 950  1850
 Wire Wire Line
-	950  2050 1450 2050
-Wire Wire Line
-	1450 2050 1850 2050
+	950  2050 1850 2050
 Connection ~ 1450 2050
 Text GLabel 1550 1050 1    60   Input ~ 0
@@
 	1550 1350 1550 1050
 Wire Wire Line
-	950  1350 1450 1350
-Wire Wire Line
-	1450 1350 1550 1350
+	950  1350 1550 1350
 Wire Wire Line
 	1650 1450 1650 1050
 Wire Wire Line
-	950  1450 1450 1450
-Wire Wire Line
-	1450 1450 1650 1450
+	950  1450 1650 1450
 Connection ~ 1450 1350
 Connection ~ 1450 1450
@@
 	3900 1100 3700 1100
 Wire Wire Line
-	3450 1450 3600 1450
-Wire Wire Line
-	3600 1450 3900 1450
+	3450 1450 3900 1450
 $Comp
 L POT_TRIM RV1
@@
 	4300 2150 4900 2150
 Wire Wire Line
-	4500 1350 4900 1350
-Wire Wire Line
-	4900 1350 5100 1350
+	4500 1350 5100 1350
 Wire Wire Line
 	4900 2300 4150 2300
 Connection ~ 4900 2150
 Wire Wire Line
-	4900 1350 4900 2150
-Wire Wire Line
-	4900 2150 4900 2300
+	4900 1350 4900 2300
 Connection ~ 3600 1450
 Text GLabel 3000 1450 0    60   Input ~ 0
@@
 $EndComp
 Wire Wire Line
-	6550 3600 6700 3600
-Wire Wire Line
-	6700 3600 6800 3600
+	6550 3600 6800 3600
 Wire Wire Line
 	6550 3600 6550 3500
@@
 	8000 2050 8000 1950
 Wire Wire Line
-	7100 2050 7550 2050
-Wire Wire Line
-	7550 2050 8000 2050
+	7100 2050 8000 2050
 Wire Wire Line
 	7100 2050 7100 1950
@@
 	7100 900  7100 1000
 Wire Wire Line
-	7100 1300 7100 1400
-Wire Wire Line
-	7100 1400 7100 1550
+	7100 1300 7100 1550
 $Comp
 L GND #PWR012
@@
 	8450 1900 8450 1750
 Wire Wire Line
-	8300 1750 8450 1750
-Wire Wire Line
-	8450 1750 8950 1750
+	8300 1750 8950 1750
 Text GLabel 6600 1750 0    60   Input ~ 0
 VIN
@@
 	7550 3200 7550 2800
 Wire Wire Line
-	6950 3200 7300 3200
-Wire Wire Line
-	7300 3200 7550 3200
+	6950 3200 7550 3200
 Wire Wire Line
 	7300 3200 7300 2450
@@
 	7100 1400 6050 1400
 Wire Wire Line
-	6050 1400 6050 2450
-Wire Wire Line
-	6050 2450 6050 3100
+	6050 1400 6050 3100
 Wire Wire Line
 	6050 3100 6350 3100
@@
 	8000 1500 8700 1500
 Wire Wire Line
-	8700 1500 8700 1950
-Wire Wire Line
-	8700 1950 8700 2700
+	8700 1500 8700 2700
 Wire Wire Line
 	8700 1950 8950 1950
@@
 	9950 2700 9950 1850
 Wire Wire Line
-	9550 1850 9950 1850
-Wire Wire Line
-	9950 1850 10150 1850
+	9550 1850 10150 1850
 Wire Wire Line
 	9050 2700 9050 2850
@@
 	1900 5600 2000 5600
 Wire Wire Line
-	2000 5500 2000 5600
-Wire Wire Line
-	2000 5600 2000 5750
+	2000 5500 2000 5750
 Wire Wire Line
 	2000 5500 2500 5500
@@
 Connection ~ 2000 5600
 Wire Wire Line
-	2400 4600 2400 5300
-Wire Wire Line
-	2400 5300 2400 5750
+	2400 4600 2400 5750
 Connection ~ 2400 5300
 $Comp
@@
 $EndComp
 Wire Wire Line
-	2000 6800 2200 6800
-Wire Wire Line
-	2200 6800 2400 6800
+	2000 6800 2400 6800
 Wire Wire Line
 	2400 6800 2400 6650
@@
 	2650 4600 2400 4600
 Wire Wire Line
-	2950 4600 3400 4600
-Wire Wire Line
-	3400 4600 3550 4600
+	2950 4600 3550 4600
 Wire Wire Line
 	3400 4600 3400 5400
 Wire Wire Line
-	3100 5400 3400 5400
-Wire Wire Line
-	3400 5400 3950 5400
+	3100 5400 3950 5400
 Text GLabel 3550 4600 2    60   Input ~ 0
 Tri-SMPL
@@
 	3900 6200 4250 6200
 Wire Wire Line
-	3900 5600 3900 5750
-Wire Wire Line
-	3900 5750 3900 6200
+	3900 5600 3900 6200
 Wire Wire Line
 	3900 5600 3950 5600
@@
 	4550 6200 4900 6200
 Wire Wire Line
-	4900 5500 4900 6200
-Wire Wire Line
-	4900 6200 4900 6450
-Wire Wire Line
-	4550 5500 4900 5500
-Wire Wire Line
-	4900 5500 5050 5500
+	4900 5500 4900 6450
+Wire Wire Line
+	4550 5500 5050 5500
 $Comp
 L R R16
@@
 $EndComp
 Wire Wire Line
-	4150 4950 4300 4950
-Wire Wire Line
-	4300 4950 4350 4950
+	4150 4950 4350 4950
 Wire Wire Line
 	4150 4950 4150 5200
@@
 	7900 5050 7900 4500
 Wire Wire Line
-	7550 4500 7900 4500
-Wire Wire Line
-	7900 4500 8050 4500
+	7550 4500 8050 4500
 Wire Wire Line
 	6950 5700 6950 6150
@@
 	7900 6150 7900 5600
 Wire Wire Line
-	7550 5600 7900 5600
-Wire Wire Line
-	7900 5600 8050 5600
+	7550 5600 8050 5600
 $Comp
 L GND #PWR021
@@
 $EndComp
 Wire Wire Line
-	4600 1050 4650 1050
-Wire Wire Line
-	4650 1050 4700 1050
+	4600 1050 4700 1050
 Connection ~ 4650 1050
 $Comp
@@
 Connection ~ 6700 3600
 Wire Wire Line
-	7100 3600 7150 3600
-Wire Wire Line
-	7150 3600 7200 3600
+	7100 3600 7200 3600
 Connection ~ 7150 3600
 Wire Wire Line
@@
 	10000 1450 9950 1450
 Wire Wire Line
-	9550 1450 9600 1450
-Wire Wire Line
-	9600 1450 9650 1450
+	9550 1450 9650 1450
 Connection ~ 9600 1450
 $Comp
@@
 F 0 "C12" H 10318 5146 50  0000 L CNN
 F 1 "100uf" H 10318 5055 50  0000 L CNN
-F 2 "Capacitors_THT:CP_Radial_D6.3mm_P2.50mm" H 10238 4950 50  0001 C CNN
+F 2 "Capacitors_THT:CP_Radial_D8.0mm_P3.50mm" H 10238 4950 50  0001 C CNN
 F 3 "" H 10200 5100 50  0001 C CNN
 	1    10200 5100
@@
 F 0 "C13" H 10768 5146 50  0000 L CNN
 F 1 "100uf" H 10768 5055 50  0000 L CNN
-F 2 "Capacitors_THT:CP_Radial_D6.3mm_P2.50mm" H 10688 4950 50  0001 C CNN
+F 2 "Capacitors_THT:CP_Radial_D8.0mm_P3.50mm" H 10688 4950 50  0001 C CNN
 F 3 "" H 10650 5100 50  0001 C CNN
 	1    10650 5100
@@
 $EndComp
 Wire Wire Line
-	10200 5300 10400 5300
-Wire Wire Line
-	10400 5300 10650 5300
-Wire Wire Line
-	10650 5300 10900 5300
+	10200 5300 10900 5300
 Wire Wire Line
 	10200 5300 10200 5250
@@
 F 0 "C14" H 10518 5546 50  0000 L CNN
 F 1 "100uf" H 10518 5455 50  0000 L CNN
-F 2 "Capacitors_THT:CP_Radial_D6.3mm_P2.50mm" H 10438 5350 50  0001 C CNN
+F 2 "Capacitors_THT:CP_Radial_D8.0mm_P3.50mm" H 10438 5350 50  0001 C CNN
 F 3 "" H 10400 5500 50  0001 C CNN
 	1    10400 5500
@@
 C9's value has a drastic\neffect on the VCO's frequency.
 Wire Wire Line
-	2700 5800 2750 5800
-Wire Wire Line
-	2750 5800 2850 5800
+	2700 5800 2850 5800
 Wire Wire Line
 	3550 5750 3500 5750
 Wire Wire Line
-	3500 5300 3500 5750
-Wire Wire Line
-	3500 5750 3500 5850
+	3500 5300 3500 5850
 Wire Wire Line
 	3500 6150 3500 6200
@@
 	3500 4950 3500 5000
 Wire Wire Line
-	9150 1250 9150 1450
-Wire Wire Line
-	9150 1450 9150 1550
+	9150 1250 9150 1550
 Wire Wire Line
 	9250 1450 9150 1450
@@
 	9950 2700 9450 2700
 Wire Wire Line
-	8700 2700 9050 2700
-Wire Wire Line
-	9050 2700 9150 2700
+	8700 2700 9150 2700
 $Comp
 L R R13
@@
 $EndComp
 Wire Wire Line
-	2150 5300 2400 5300
-Wire Wire Line
-	2400 5300 2500 5300
+	2150 5300 2500 5300
 $Comp
 L POT_TRIM RV4
@@
 RV1 is exponential product control.\nRV2 is product control.\nRV3 and RV4 are sum controls.
 Wire Wire Line
-	3600 1450 3600 1800
-Wire Wire Line
-	3600 1800 3600 2150
+	3600 1450 3600 2150
 Wire Wire Line
 	3600 2150 4000 2150
@@
 $EndComp
 Wire Wire Line
-	1150 3450 1150 3850
-Wire Wire Line
-	1150 3850 1150 3900
+	1150 3450 1150 3900
 Wire Wire Line
 	1150 3850 1200 3850
@@
 $EndComp
 Wire Wire Line
-	2850 6750 3000 6750
-Wire Wire Line
-	3000 6750 3650 6750
-Wire Wire Line
-	3650 6750 3750 6750
+	2850 6750 3750 6750
 Connection ~ 3650 6750
 $Comp
@@
 	1750 5200 1550 5200
 Wire Wire Line
-	1550 5200 1550 5400
-Wire Wire Line
-	1550 5400 1550 5600
+	1550 5200 1550 5600
 Wire Wire Line
 	1550 5600 1600 5600

Commit message: Delete old files and start over
Parts:
- removed C1, C10, C11, C15, C2, C3, C4, C6, C7, C8: 100nf, Capacitors_THT:C_Disc_D5.0mm_W2.5mm_P2.50mm, symbol C
- removed C12, C13, C14: 100uf, Capacitors_THT:CP_Radial_D8.0mm_P3.50mm, symbol CP
- removed C5: 1nf, Capacitors_THT:C_Disc_D3.8mm_W2.6mm_P2.50mm, symbol C
- removed C9: 4nf, Capacitors_THT:C_Rect_L7.0mm_W3.5mm_P2.50mm_P5.00mm, symbol C
- removed J1: CONN_02X08, Pin_Headers:Pin_Header_Straight_2x08_Pitch2.54mm, symbol CONN_02X08
- removed J2, J3, J4, J5: PJ301M-12, Eurocad:PJ301M-12, symbol PJ301M-12
- removed Q1, Q2, Q3, Q5, Q6: 2N3904, TO_SOT_Packages_THT:TO-92_Inline_Wide, symbol 2N3904
- removed Q4: 2N3906, TO_SOT_Packages_THT:TO-92_Inline_Wide, symbol 2N3906
- removed R1: 1M, Resistors_THT:R_Axial_DIN0207_L6.3mm_D2.5mm_P10.16mm_Horizontal, symbol R
- removed R10, R11, R12, R13: 50k, Resistors_THT:R_Axial_DIN0207_L6.3mm_D2.5mm_P10.16mm_Horizontal, symbol R
- removed R14, R15, R16, R17, R2, R3, R8, R9: 100k, Resistors_THT:R_Axial_DIN0207_L6.3mm_D2.5mm_P10.16mm_Horizontal, symbol R
- removed R18, R4: 10k, Resistors_THT:R_Axial_DIN0207_L6.3mm_D2.5mm_P10.16mm_Horizontal, symbol R
- removed R5, R7: 1k, Resistors_THT:R_Axial_DIN0207_L6.3mm_D2.5mm_P10.16mm_Horizontal, symbol R
- removed RV1, RV3, RV4: 10k, Potentiometers:Potentiometer_Trimmer_Bourns_3296Y, symbol POT_TRIM
- removed RV2: 100k, Potentiometers:Potentiometer_Trimmer_Bourns_3296Y, symbol POT_TRIM
- removed RV5: 10k, Potentiometers:Potentiometer_Alps_RK09L_Sleve_Single_Horizontal_Custom, symbol POT
- removed U1, U2, U3, U4, U5, U6, U7: LM741, Housings_DIP:DIP-8_W7.62mm, symbol LM741
Connections:
- net labels removed: +12V, +5V, -12VA, CV, CV1, Exp-CV, GND, Gate, Gate1, Sqr-SMPL, Square, Tri-SMPL, Triangle, VIN
- wire segments 168 -> 0
- no-connect marks 17 -> 0
Other:
- note removed: "C9's value has a drastic\neffect on the VCO's frequency."
- note removed: "Exponential Converter"
- note removed: "Input Amp"
- note removed: "Output Buffers"
- note removed: "Pitch control pot."
- note removed: "RV1 is exponential product control.\nRV2 is product control.\nRV3 and RV4 are sum controls."
- note removed: "Thermal Bonding"
- note removed: "VCO"

Commit message: Begin working on ports
Changed lines of the file:
@@
 EESchema Schematic File Version 4
+LIBS:analog-synth-1-cache
 EELAYER 26 0
 EELAYER END
@@
 $EndDescr
 $Sheet
-S 1200 1200 1150 550
+S 1350 1400 1150 550
 U 5C85AB83
 F0 "Analog Synth 1 Ports" 50
